File: H_bridge_PCB/H_bridge_PCB.kicad_pcb (KiCad board)
At the start: 2 copper layers, 68.6 x 53.3 mm, 15 parts, among them J1 PWR IN, J2 CH L, J3 CH R, J4 Bluetooth module connector, J5 PWR IN jumper, U1 DRV8844PWPR, U2 MC79M05_TO252

Commit message: yah
Parts:
- moved C7 0.87 mm to (114.5, 120.5)
Changed lines of the file:
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@@
   (net 52 "Net-(C1-Pad1)")
   (footprint "Capacitor_THT:C_Axial_L19.0mm_D8.0mm_P25.00mm_Horizontal" (layer "F.Cu")
-    (at 114.554 119.634)
+    (at 114.5 120.5)
     (descr "C, Axial series, Axial, Horizontal, pin pitch=25mm, , length*diameter=19*8.0mm^2, http://cdn-reichelt.de/documents/datenblatt/B300/STYROFLEX.pdf")
     (tags "C Axial series Axial Horizontal pin pitch 25mm  length 19mm diameter 8.0mm")
@@
     )
   )
+  (gr_rect (start 117.5 98) (end 135.5 116) (layer "F.SilkS") (width 0.15) (fill none))
   (segment (start 122.396 110.255) (end 123.465 110.255) (width 0.25) (layer "B.Cu") (net 1))
   (segment (start 121.285 111.366) (end 122.396 110.255) (width 0.25) (layer "B.Cu") (net 1))
   (segment (start 148.85 121.108) (end 146.935 121.108) (width 0.25) (layer "F.Cu") (net 2))
+  (segment (start 140.366 119.634) (end 139.5 120.5) (width 0.25) (layer "F.Cu") (net 2))
+  (segment (start 145.461 119.634) (end 140.366 119.634) (width 0.25) (layer "F.Cu") (net 2))
   (segment (start 150.355 124.528) (end 148.85 123.023) (width 0.25) (layer "F.Cu") (net 2))
-  (segment (start 145.461 119.634) (end 139.554 119.634) (width 0.25) (layer "F.Cu") (net 2))
   (segment (start 146.05 120.223) (end 145.461 119.634) (width 0.25) (layer "F.Cu") (net 2))
   (segment (start 148.85 123.023) (end 148.85 121.108) (width 0.25) (layer "F.Cu") (net 2))
   (segment (start 146.935 121.108) (end 146.05 120.223) (width 0.25) (layer "F.Cu") (net 2))
-  (segment (start 137.994 119.634) (end 129.265 110.905) (width 0.25) (layer "B.Cu") (net 2))
-  (segment (start 139.554 119.634) (end 137.994 119.634) (width 0.25) (layer "B.Cu") (net 2))
-  (segment (start 140.535 131.0815) (end 140.535 120.615) (width 0.25) (layer "B.Cu") (net 2))
-  (segment (start 140.535 120.615) (end 139.554 119.634) (width 0.25) (layer "B.Cu") (net 2))
-  (segment (start 128.778 119.634) (end 114.554 119.634) (width 0.25) (layer "F.Cu") (net 3))
-  (segment (start 143.002 113.157) (end 135.255 113.157) (width 0.25) (layer "F.Cu") (net 3))
-  (segment (start 135.255 113.157) (end 128.778 119.634) (width 0.25) (layer "F.Cu") (net 3))
+  (segment (start 139.5 120.5) (end 138.86 120.5) (width 0.25) (layer "B.Cu") (net 2))
+  (segment (start 140.535 121.535) (end 139.5 120.5) (width 0.25) (layer "B.Cu") (net 2))
+  (segment (start 138.86 120.5) (end 129.265 110.905) (width 0.25) (layer "B.Cu") (net 2))
+  (segment (start 140.535 131.0815) (end 140.535 121.535) (width 0.25) (layer "B.Cu") (net 2))
+  (segment (start 132.866 119.634) (end 115.366 119.634) (width 0.25) (layer "F.Cu") (net 3))
+  (segment (start 143.002 113.157) (end 139.343 113.157) (width 0.25) (layer "F.Cu") (net 3))
+  (segment (start 115.366 119.634) (end 114.5 120.5) (width 0.25) (layer "F.Cu") (net 3))
+  (segment (start 139.343 113.157) (end 132.866 119.634) (width 0.25) (layer "F.Cu") (net 3))
   (via (at 113.03 114.3) (size 0.8) (drill 0.4) (layers "F.Cu" "B.Cu") (free) (net 3))
   (via (at 114.3 114.3) (size 0.8) (drill 0.4) (layers "F.Cu" "B.Cu") (free) (net 3))
